File: PCB/Edge_Atmos_PCB.kicad_sch (KiCad schematic)
At the start: 0 parts

Commit message: Adding box structure to display library
Parts:
- added J1: AHT10, Connector_PinSocket_2.54mm:PinSocket_1x04_P2.54mm_Vertical, symbol Connector_Generic:Conn_01x04
- added J2: BMP280, Connector_PinSocket_2.54mm:PinSocket_1x06_P2.54mm_Vertical, symbol Connector_Generic:Conn_01x06
- added J3: W25Q32, Connector_PinSocket_2.54mm:PinSocket_1x06_P2.54mm_Vertical, symbol Connector_Generic:Conn_01x06
- added J4: STM32F103C8T6_1, Connector_PinSocket_2.54mm:PinSocket_1x20_P2.54mm_Vertical, symbol Connector_Generic:Conn_01x20
- added J5: STM32F103C8T6_2, Connector_PinSocket_2.54mm:PinSocket_1x20_P2.54mm_Vertical, symbol Connector_Generic:Conn_01x20
- added J6: TFT, Connector_PinSocket_2.54mm:PinSocket_1x14_P2.54mm_Vertical, symbol Connector_Generic:Conn_01x14
- added J7: Conn_01x04, Connector_PinSocket_2.54mm:PinSocket_1x04_P2.54mm_Vertical, symbol Connector_Generic:Conn_01x04
Connections:
- new net GND: J1.2 (Pin_2), J2.2 (Pin_2), J3.4 (Pin_4), J4.19 (Pin_19), J6.2 (Pin_2)
- new net MEM_CS: J3.2 (Pin_2), J5.12 (Pin_12)
- new net MISO1: J3.3 (Pin_3), J5.10 (Pin_10), J6.9 (Pin_9)
- new net MOSI1: J3.6 (Pin_6), J5.9 (Pin_9), J6.6 (Pin_6)
- new net SCK1: J3.5 (Pin_5), J5.11 (Pin_11), J6.7 (Pin_7)
- new net SCL1: J1.3 (Pin_3), J2.3 (Pin_3), J4.14 (Pin_14)
- new net SDA1: J1.4 (Pin_4), J2.4 (Pin_4), J4.15 (Pin_15)
- new net TFT_CS: J5.13 (Pin_13), J6.3 (Pin_3)
- new net TFT_DC: J5.15 (Pin_15), J6.5 (Pin_5)
- new net TFT_LED: J5.16 (Pin_16), J6.8 (Pin_8)
- new net TFT_RST: J5.14 (Pin_14), J6.4 (Pin_4)
- new net VIN: J1.1 (Pin_1), J2.1 (Pin_1), J3.1 (Pin_1), J4.20 (Pin_20), J6.1 (Pin_1)
- no-connect marks 0 -> 39
Other:
- title: (none) -> Edge Atmos
